Commit message: Clean up codebase to a minimal, defined scope
GangubAI is now: wake word -> voice Q&A over course slides (RAG, Groq),
timer/pomodoro overlays, voice-driven movement and wander mode, and an
animated Pygame face. Runs on Raspberry Pi 5 (lgpio) or in Gazebo.

Removed:
- push-to-talk, text chat CLI, calculator tool, WAV test mode
- ROS emotion bridge (face now listens on UDP only)
- unused optimized/persistent transcribers, config_optimized, profiler
- duplicate face assets folder and duplicate launcher
- motor demo mode, optical-flow stuck check, Range cliff path, status topics
- RPi.GPIO fallback, generated-face fallback, module self-test CLIs

Changed:
- ai/robot.py: single place for /motor_command and /wander_mode publishing
- graph.py: keep only RAG + movement keyword fallbacks, temperature 0.2,
  and fix a loop where a forced move could repeat after the tool ran
- RAG indexes every PPTX/PDF in ai/chatbot/Unit1
- tts.py: two explicit outputs (aplay for MAX98357A, sounddevice) chosen
  by TTS_USE_APLAY
- wake_word.py: current OpenWakeWord API only
- requirements.txt filled in, README rewritten for the actual project

Co-Authored-By: Claude Opus 5.5 <noreply@anthropic.com>

File: ros2_ws/src/gangubai_description/urdf/gangubai.urdf (robot description, URDF)
Before this commit: robot gangubai, 8 links, 7 joints
Links:
- removed link optical_sensor_link
Joints:
- removed joint optical_joint
